File: kicad/PhonePiHat/PhonePiHat.kicad_pcb (KiCad board)
At the start: 2 copper layers, 31.8 x 67 mm, 12 parts, among them J1 Raspberry_Pi_4, J2 Screw_Terminal_01x13, Q1 IRF540N

Commit message: v2 board
Parts:
- J1: moved to B.Cu
- moved J2 73.5 mm to (31.5, 44.0), turned to -90 degrees
- moved Q1 50.1 mm to (40.0, 50.1)
- moved R4 33.3 mm to (38.5, 76.2)
- moved R9 33.3 mm to (38.5, 91.9)
- moved R3 33.3 mm to (38.5, 73.0)
- moved R5 33.3 mm to (38.5, 79.3)
- moved R6 33.3 mm to (38.5, 82.5)
- moved R7 33.3 mm to (38.5, 85.6)
- moved R8 33.3 mm to (38.5, 88.8)
- moved R10 30.0 mm to (38.6, 97.3)
- moved R1 27.3 mm to (38.1, 56.0)
- moved J1 13.7 mm to (45.2, 48.9), turned to 180 degrees
Connections:
- J1 pad 14: Net-(J2-Pin_4) -> Net-(Q1-S)
- J1 pad 20: Net-(J2-Pin_4) -> Net-(Q1-S)
- J1 pad 25: Net-(J2-Pin_4) -> Net-(Q1-S)
- J1 pad 30: Net-(J2-Pin_4) -> Net-(Q1-S)
- J1 pad 34: Net-(J2-Pin_4) -> Net-(Q1-S)
- J1 pad 39: Net-(J2-Pin_4) -> Net-(Q1-S)
- J1 pad 6: Net-(J2-Pin_4) -> Net-(Q1-S)
- J1 pad 9: Net-(J2-Pin_4) -> Net-(Q1-S)
- Q1 pad 3: Net-(J2-Pin_4) -> Net-(Q1-S)
- R1 pad 2: Net-(J2-Pin_4) -> Net-(Q1-S)
- R10 pad 2: Net-(J2-Pin_4) -> Net-(Q1-S)
- R3 pad 2: Net-(J2-Pin_4) -> Net-(Q1-S)
- R4 pad 2: Net-(J2-Pin_4) -> Net-(Q1-S)
- R5 pad 2: Net-(J2-Pin_4) -> Net-(Q1-S)
- R6 pad 2: Net-(J2-Pin_4) -> Net-(Q1-S)
- R7 pad 2: Net-(J2-Pin_4) -> Net-(Q1-S)
- R8 pad 2: Net-(J2-Pin_4) -> Net-(Q1-S)
- R9 pad 2: Net-(J2-Pin_4) -> Net-(Q1-S)
Routing:
- net Net-(Q1-S): track 0.00 -> 101.5 mm
- net Net-(J2-Pin_4): track 129.9 -> 44.0 mm, vias 0 -> 1
- net Net-(J1-GPIO20/SPI1_MOSI/PCM_DIN/PWM1): track 65.8 -> 21.5 mm, vias 2 -> 0
- net Net-(J1-GPIO17/SPI1_~{CE1}): track 59.7 -> 16.0 mm
- net Net-(J2-Pin_2): track 63.3 -> 20.1 mm, vias 1 -> 0
- net Net-(J1-GPIO19/SPI1_MISO/PCM_FS): track 62.3 -> 20.9 mm
- net Net-(J1-GPIO21/SPI1_SCLK/PCM_DOUT): track 20.4 -> 59.1 mm, vias 0 -> 1
- net Net-(J1-GPIO26/SDIO_DAT2): track 51.0 -> 22.9 mm
- net Net-(J1-GPIO22/SDIO_CLK): track 44.2 -> 23.4 mm
- net Net-(J1-GPIO23/SDIO_CMD): track 42.1 -> 22.4 mm
- net Net-(J1-GPIO25/SDIO_DAT1): track 31.1 -> 20.9 mm, vias 1 -> 0
- net Net-(J1-GPIO24/SDIO_DAT0): track 34.1 -> 24.3 mm
- net Net-(J1-GPIO27/SDIO_DAT3): track 27.3 -> 36.9 mm, vias 1 -> 0
- net Net-(J2-Pin_1): track 17.6 -> 9.97 mm
Other:
- board size 31.8 x 67 mm -> 33 x 67.4 mm
- board text added: "10k"
- board text added: "1k"
- board text added: "AJS v0.1"
- board text added: "PhonePiHat"
